Commit message: Update test srdf/urdf files

File: boostXmlParser/test.urdf (robot description, URDF)
Before this commit: robot A02L-M1, 2 links, 0 joints
Joints:
- added joint joint1: type revolute, parent base_link, child link1, origin xyz=0.0 0.0 0.155 rpy=0.0 0.0 -3.141592653589793, axis 0 0 1, limit lower=-2.7925 upper=2.7925 effort=123 velocity=2.0944
